Commit message: Added ability to train dynamics-model without a specific task, made changes to try to use challenge_envs but no success, added a PPO agent but it hasn't been fully tested and is not ready to go yet

File: challenging_envs/envs/urdfs/cube/cube.urdf (robot description, URDF)
Before this commit: robot cube.urdf, 1 links, 0 joints
Links:
- link baseLink: geometry collision box size=128 .1 128; visual mesh filename=cube.obj scale=128.0 .1 128

Commit message: Added TRPO implementation

File: challenging_envs/envs/urdfs/cube/cube.urdf (robot description, URDF)
Before this commit: robot cube.urdf, 1 links, 0 joints
Links:
- link baseLink: geometry collision box size=0.1 100 1; visual mesh filename=cube.obj scale=0.1 100 1
